File: KiCad_DC_Load/Power_Supply.sch (KiCad schematic (older format))
At the start: 8 parts, among them U1 L7809

Commit message: Some footprints assigned
Parts:
- C10, C11, C8, C9: renamed from C?; footprint (none) -> Capacitor_SMD:C_0805_2012Metric
- JST_Power1: renamed from JST_Power; footprint Connector_JST:JST_EH_B2B-EH-A_1x02_P2.50mm_Vertical -> Connector_JST:JST_PH_B2B-PH-K_1x02_P2.00mm_Vertical
- JST_Power_Button1: renamed from JST_Power_Button; footprint (none) -> Connector_JST:JST_PH_B4B-PH-K_1x04_P2.00mm_Vertical
- gave numbers to parts that had none: 1
- renumbered U1 to U3
Changed lines of the file:
@@
 Sheet 4 6
 Title "Power Supply"
-Date ""
-Rev ""
+Date "2021-06-16"
+Rev "v01"
 Comp ""
 Comment1 ""
 Comment2 ""
 Comment3 ""
-Comment4 "HappyDonuts"
+Comment4 "Author: HappyDonuts"
 $EndDescr
 $Comp
-L Regulator_Linear:L7809 U1
+L Regulator_Linear:L7809 U3
 U 1 1 5FD2AD92
 P 3350 1500
-F 0 "U1" H 3350 1742 50  0000 C CNN
+F 0 "U3" H 3350 1742 50  0000 C CNN
 F 1 "L7809" H 3350 1651 50  0000 C CNN
 F 2 "" H 3375 1350 50  0001 L CIN
@@
 $EndComp
 $Comp
-L Device:C C?
+L Device:C C8
 U 1 1 5FD2C09B
 P 2850 1700
-F 0 "C?" H 2965 1746 50  0000 L CNN
+F 0 "C8" H 2965 1746 50  0000 L CNN
 F 1 "330n" H 2965 1655 50  0000 L CNN
-F 2 "" H 2888 1550 50  0001 C CNN
+F 2 "Capacitor_SMD:C_0805_2012Metric" H 2888 1550 50  0001 C CNN
 F 3 "~" H 2850 1700 50  0001 C CNN
 	1    2850 1700
@@
 $EndComp
 $Comp
-L Device:C C?
+L Device:C C10
 U 1 1 5FD2C83F
 P 3850 1700
-F 0 "C?" H 3965 1746 50  0000 L CNN
+F 0 "C10" H 3965 1746 50  0000 L CNN
 F 1 "100n" H 3965 1655 50  0000 L CNN
-F 2 "" H 3888 1550 50  0001 C CNN
+F 2 "Capacitor_SMD:C_0805_2012Metric" H 3888 1550 50  0001 C CNN
 F 3 "~" H 3850 1700 50  0001 C CNN
 	1    3850 1700
@@
 	3850 1900 3850 1850
 $Comp
-L power:GND #PWR0110
+L power:GND #PWR021
 U 1 1 5FD2D1EB
 P 3350 1950
-F 0 "#PWR0110" H 3350 1700 50  0001 C CNN
+F 0 "#PWR021" H 3350 1700 50  0001 C CNN
 F 1 "GND" H 3355 1777 50  0000 C CNN
 F 2 "" H 3350 1950 50  0001 C CNN
@@
 Connection ~ 3850 1500
 $Comp
-L Regulator_Linear:L7805 U?
+L Regulator_Linear:L7805 U4
 U 1 1 60C35BD0
 P 3350 2600
-F 0 "U?" H 3350 2842 50  0000 C CNN
+F 0 "U4" H 3350 2842 50  0000 C CNN
 F 1 "L7805" H 3350 2751 50  0000 C CNN
 F 2 "" H 3375 2450 50  0001 L CIN
@@
 $EndComp
 $Comp
-L Device:C C?
+L Device:C C9
 U 1 1 60C37A92
 P 2850 2800
-F 0 "C?" H 2965 2846 50  0000 L CNN
+F 0 "C9" H 2965 2846 50  0000 L CNN
 F 1 "330n" H 2965 2755 50  0000 L CNN
-F 2 "" H 2888 2650 50  0001 C CNN
+F 2 "Capacitor_SMD:C_0805_2012Metric" H 2888 2650 50  0001 C CNN
 F 3 "~" H 2850 2800 50  0001 C CNN
 	1    2850 2800
@@
 $EndComp
 $Comp
-L Device:C C?
+L Device:C C11
 U 1 1 60C38101
 P 3850 2800
-F 0 "C?" H 3965 2846 50  0000 L CNN
+F 0 "C11" H 3965 2846 50  0000 L CNN
 F 1 "100n" H 3965 2755 50  0000 L CNN
-F 2 "" H 3888 2650 50  0001 C CNN
+F 2 "Capacitor_SMD:C_0805_2012Metric" H 3888 2650 50  0001 C CNN
 F 3 "~" H 3850 2800 50  0001 C CNN
 	1    3850 2800
@@
 $EndComp
 $Comp
-L power:GND #PWR?
+L power:GND #PWR022
 U 1 1 60C384D4
 P 3350 3050
-F 0 "#PWR?" H 3350 2800 50  0001 C CNN
+F 0 "#PWR022" H 3350 2800 50  0001 C CNN
 F 1 "GND" H 3355 2877 50  0000 C CNN
 F 2 "" H 3350 3050 50  0001 C CNN
@@
 Connection ~ 2850 2600
 $Comp
-L power:GND #PWR?
+L power:GND #PWR019
 U 1 1 60C1375B
 P 1400 2000
-F 0 "#PWR?" H 1400 1750 50  0001 C CNN
+F 0 "#PWR019" H 1400 1750 50  0001 C CNN
 F 1 "GND" H 1405 1827 50  0000 C CNN
 F 2 "" H 1400 2000 50  0001 C CNN
@@
 $EndComp
 $Comp
-L Connector_Generic:Conn_01x04 JST_Power_Button
+L Connector_Generic:Conn_01x04 JST_Power_Button1
 U 1 1 60C5CD8C
 P 1950 1800
-F 0 "JST_Power_Button" H 2030 1792 50  0000 L CNN
+F 0 "JST_Power_Button1" H 2030 1792 50  0000 L CNN
 F 1 "Conn_01x04" H 2030 1701 50  0000 L CNN
-F 2 "" H 1950 1800 50  0001 C CNN
+F 2 "Connector_JST:JST_PH_B4B-PH-K_1x04_P2.00mm_Vertical" H 1950 1800 50  0001 C CNN
 F 3 "~" H 1950 1800 50  0001 C CNN
 	1    1950 1800
@@
 $EndComp
 $Comp
-L power:GND #PWR?
+L power:GND #PWR020
 U 1 1 60C61B49
 P 1750 2000
-F 0 "#PWR?" H 1750 1750 50  0001 C CNN
+F 0 "#PWR020" H 1750 1750 50  0001 C CNN
 F 1 "GND" H 1755 1827 50  0000 C CNN
 F 2 "" H 1750 2000 50  0001 C CNN
@@
 $EndComp
 $Comp
-L Connector_Generic:Conn_01x02 JST_Power
+L Connector_Generic:Conn_01x02 JST_Power1
 U 1 1 60C0D512
 P 1200 1900
-F 0 "JST_Power" H 1118 2117 50  0000 C CNN
+F 0 "JST_Power1" H 1118 2117 50  0000 C CNN
 F 1 "Conn_01x02" H 1118 2026 50  0000 C CNN
-F 2 "Connector_JST:JST_EH_B2B-EH-A_1x02_P2.50mm_Vertical" H 1200 1900 50  0001 C CNN
+F 2 "Connector_JST:JST_PH_B2B-PH-K_1x02_P2.00mm_Vertical" H 1200 1900 50  0001 C CNN
 F 3 "~" H 1200 1900 50  0001 C CNN
 	1    1200 1900
