File: KiCad_DC_Load/Load_Circuit.sch (KiCad schematic (older format))
At the start: 34 parts, among them K1 G5LE-1, K2 G5LE-1, Q1 Q_NMOS_GDS, U1 LMC6482, U2 GS8552

Commit message: Power supply and connectors
Parts:
- added C? (x4): 100n, symbol Device:C
Connections:
- net GND: now also C?.2, C?.2
- net v_5: now also C?.1
- net v_9: now also C?.1, C?.1, C?.1; no longer R?.1
- net v_load: now reaches K1.1
- net v_load: now also R?.1
Other:
- moved on the sheet: D?, K1, Q?, R?
Changed lines of the file:
@@
 Connection ~ 6400 4450
-$Comp
-L Relay:G5LE-1 K1
-U 1 1 5FD31D61
-P 5600 2300
-F 0 "K1" H 5170 2254 50  0000 R CNN
-F 1 "G5LE-1" H 5170 2345 50  0000 R CNN
-F 2 "Relay_THT:Relay_SPDT_Omron-G5LE-1" H 6050 2250 50  0001 L CNN
-F 3 "http://www.omron.com/ecb/products/pdf/en-g5le.pdf" H 5600 2300 50  0001 C CNN
-	1    5600 2300
-	-1   0    0    1
-$EndComp
 $Comp
 L Device:D D1
@@
 Wire Wire Line
 	5300 3150 5300 3300
-Wire Wire Line
-	5300 2850 5300 2600
 $Comp
 L Diode:1N4007 D?
 U 1 1 5FD394CC
-P 6400 2300
-F 0 "D?" V 6354 2380 50  0000 L CNN
-F 1 "1N4007" V 6445 2380 50  0000 L CNN
-F 2 "Diode_THT:D_DO-41_SOD81_P10.16mm_Horizontal" H 6400 2125 50  0001 C CNN
-F 3 "http://www.vishay.com/docs/88503/1n4001.pdf" H 6400 2300 50  0001 C CNN
-	1    6400 2300
+P 6400 2550
+F 0 "D?" V 6354 2630 50  0000 L CNN
+F 1 "1N4007" V 6445 2630 50  0000 L CNN
+F 2 "Diode_THT:D_DO-41_SOD81_P10.16mm_Horizontal" H 6400 2375 50  0001 C CNN
+F 3 "http://www.vishay.com/docs/88503/1n4001.pdf" H 6400 2550 50  0001 C CNN
+	1    6400 2550
 	0    1    1    0
 $EndComp
 Wire Wire Line
-	5800 1950 6400 1950
-Wire Wire Line
-	6400 1950 6400 2150
-Wire Wire Line
-	5800 2650 6400 2650
-Wire Wire Line
-	6400 2650 6400 2450
-Wire Wire Line
-	6400 2650 6400 2900
-Connection ~ 6400 2650
+	5800 2200 6400 2200
+Wire Wire Line
+	6400 2200 6400 2400
+Wire Wire Line
+	5800 2900 6400 2900
+Wire Wire Line
+	6400 2900 6400 2700
+Wire Wire Line
+	6400 2900 6400 3150
+Connection ~ 6400 2900
 $Comp
 L power:GND #PWR0108
 U 1 1 5FD394E6
-P 6400 3500
-F 0 "#PWR0108" H 6400 3250 50  0001 C CNN
-F 1 "GND" H 6405 3327 50  0000 C CNN
-F 2 "" H 6400 3500 50  0001 C CNN
-F 3 "" H 6400 3500 50  0001 C CNN
-	1    6400 3500
+P 6400 3750
+F 0 "#PWR0108" H 6400 3500 50  0001 C CNN
+F 1 "GND" H 6405 3577 50  0000 C CNN
+F 2 "" H 6400 3750 50  0001 C CNN
+F 3 "" H 6400 3750 50  0001 C CNN
+	1    6400 3750
 	-1   0    0    -1
 $EndComp
@@
 L Device:R R?
 U 1 1 5FD394F0
-P 6750 3350
-F 0 "R?" H 6680 3304 50  0000 R CNN
-F 1 "100k" H 6680 3395 50  0000 R CNN
-F 2 "" V 6680 3350 50  0001 C CNN
-F 3 "~" H 6750 3350 50  0001 C CNN
-	1    6750 3350
+P 6750 3600
+F 0 "R?" H 6680 3554 50  0000 R CNN
+F 1 "100k" H 6680 3645 50  0000 R CNN
+F 2 "" V 6680 3600 50  0001 C CNN
+F 3 "~" H 6750 3600 50  0001 C CNN
+	1    6750 3600
 	1    0    0    1
 $EndComp
 Wire Wire Line
-	6750 3200 6750 3100
-Wire Wire Line
-	6750 3100 6700 3100
+	6750 3450 6750 3350
+Wire Wire Line
+	6750 3350 6700 3350
 $Comp
 L power:GND #PWR0109
 U 1 1 5FD394FC
-P 6750 3500
-F 0 "#PWR0109" H 6750 3250 50  0001 C CNN
-F 1 "GND" H 6755 3327 50  0000 C CNN
-F 2 "" H 6750 3500 50  0001 C CNN
-F 3 "" H 6750 3500 50  0001 C CNN
-	1    6750 3500
-	-1   0    0    -1
-$EndComp
-Wire Wire Line
-	6400 3300 6400 3500
-Text GLabel 7250 3100 2    50   Input ~ 0
+P 6750 3750
+F 0 "#PWR0109" H 6750 3500 50  0001 C CNN
+F 1 "GND" H 6755 3577 50  0000 C CNN
+F 2 "" H 6750 3750 50  0001 C CNN
+F 3 "" H 6750 3750 50  0001 C CNN
+	1    6750 3750
+	-1   0    0    -1
+$EndComp
+Wire Wire Line
+	6400 3550 6400 3750
+Text GLabel 7250 3350 2    50   Input ~ 0
 close_circuit
 $Comp
 L Device:R R?
 U 1 1 5FD39508
-P 7000 3100
-F 0 "R?" H 6930 3054 50  0000 R CNN
-F 1 "100" H 6930 3145 50  0000 R CNN
-F 2 "" V 6930 3100 50  0001 C CNN
-F 3 "~" H 7000 3100 50  0001 C CNN
-	1    7000 3100
+P 7000 3350
+F 0 "R?" H 6930 3304 50  0000 R CNN
+F 1 "100" H 6930 3395 50  0000 R CNN
+F 2 "" V 6930 3350 50  0001 C CNN
+F 3 "~" H 7000 3350 50  0001 C CNN
+	1    7000 3350
 	0    -1   1    0
 $EndComp
 Wire Wire Line
-	6750 3100 6850 3100
-Connection ~ 6750 3100
-Wire Wire Line
-	7150 3100 7250 3100
-Text GLabel 6400 1700 1    50   Input ~ 0
+	6750 3350 6850 3350
+Connection ~ 6750 3350
+Wire Wire Line
+	7150 3350 7250 3350
+Text GLabel 6400 1950 1    50   Input ~ 0
 v_9
-Connection ~ 6400 1950
-Wire Wire Line
-	5800 2650 5800 2600
-Wire Wire Line
-	5800 2000 5800 1950
+Connection ~ 6400 2200
+Wire Wire Line
+	5800 2250 5800 2200
 Wire Wire Line
 	5700 5150 6400 5150
@@
 L Transistor_FET:2N7002 Q?
 U 1 1 60BD2568
-P 6500 3100
-F 0 "Q?" H 6705 3146 50  0000 L CNN
-F 1 "2N7002" H 6705 3055 50  0000 L CNN
-F 2 "Package_TO_SOT_SMD:SOT-23" H 6700 3025 50  0001 L CIN
-F 3 "https://www.fairchildsemi.com/datasheets/2N/2N7002.pdf" H 6500 3100 50  0001 L CNN
-	1    6500 3100
+P 6500 3350
+F 0 "Q?" H 6705 3396 50  0000 L CNN
+F 1 "2N7002" H 6705 3305 50  0000 L CNN
+F 2 "Package_TO_SOT_SMD:SOT-23" H 6700 3275 50  0001 L CIN
+F 3 "https://www.fairchildsemi.com/datasheets/2N/2N7002.pdf" H 6500 3350 50  0001 L CNN
+	1    6500 3350
 	-1   0    0    -1
 $EndComp
@@
 	-1   0    0    -1
 $EndComp
-NoConn ~ 5500 2600
+NoConn ~ 5500 2800
 $Comp
 L Device:Opamp_Dual_Generic U2
@@
 	4500 1900 4500 1850
 Wire Wire Line
-	6400 1700 6400 1850
-Wire Wire Line
 	4500 1850 4600 1850
 Wire Wire Line
 	4200 1850 4500 1850
 Connection ~ 4500 1850
-Wire Wire Line
-	4900 1850 6400 1850
-Connection ~ 6400 1850
-Wire Wire Line
-	6400 1850 6400 1950
 Wire Wire Line
 	4200 2050 4300 2050
@@
 Wire Wire Line
 	1250 2150 1250 2200
+$Comp
+L Device:C C?
+U 1 1 60C16B7D
+P 1850 2550
+F 0 "C?" H 1965 2596 50  0000 L CNN
+F 1 "100n" H 1965 2505 50  0000 L CNN
+F 2 "" H 1888 2400 50  0001 C CNN
+F 3 "~" H 1850 2550 50  0001 C CNN
+	1    1850 2550
+	1    0    0    -1
+$EndComp
+$Comp
+L Device:C C?
+U 1 1 60C17345
+P 1850 1500
+F 0 "C?" H 1965 1546 50  0000 L CNN
+F 1 "100n" H 1965 1455 50  0000 L CNN
+F 2 "" H 1888 1350 50  0001 C CNN
+F 3 "~" H 1850 1500 50  0001 C CNN
+	1    1850 1500
+	1    0    0    -1
+$EndComp
+Wire Wire Line
+	1850 1350 1850 1150
+Wire Wire Line
+	1850 1150 1250 1150
+Connection ~ 1250 1150
+Wire Wire Line
+	1250 1750 1850 1750
+Wire Wire Line
+	1850 1750 1850 1650
+Wire Wire Line
+	1250 2750 1850 2750
+Wire Wire Line
+	1850 2750 1850 2700
+Wire Wire Line
+	1250 2150 1850 2150
+Wire Wire Line
+	1850 2150 1850 2400
+Connection ~ 1250 2150
+$Comp
+L Device:C C?
+U 1 1 60C28823
+P 7000 4800
+F 0 "C?" H 7115 4846 50  0000 L CNN
+F 1 "100n" H 7115 4755 50  0000 L CNN
+F 2 "" H 7038 4650 50  0001 C CNN
+F 3 "~" H 7000 4800 50  0001 C CNN
+	1    7000 4800
+	1    0    0    -1
+$EndComp
+$Comp
+L Device:C C?
+U 1 1 60C28F02
+P 7000 2550
+F 0 "C?" H 7115 2596 50  0000 L CNN
+F 1 "100n" H 7115 2505 50  0000 L CNN
+F 2 "" H 7038 2400 50  0001 C CNN
+F 3 "~" H 7000 2550 50  0001 C CNN
+	1    7000 2550
+	1    0    0    -1
+$EndComp
+Wire Wire Line
+	6400 2200 7000 2200
+Wire Wire Line
+	7000 2200 7000 2400
+$Comp
+L power:GND #PWR?
+U 1 1 60C2E9A7
+P 7000 4950
+F 0 "#PWR?" H 7000 4700 50  0001 C CNN
+F 1 "GND" H 7005 4777 50  0000 C CNN
+F 2 "" H 7000 4950 50  0001 C CNN
+F 3 "" H 7000 4950 50  0001 C CNN
+	1    7000 4950
+	-1   0    0    -1
+$EndComp
+$Comp
+L power:GND #PWR?
+U 1 1 60C2EE08
+P 7000 2700
+F 0 "#PWR?" H 7000 2450 50  0001 C CNN
+F 1 "GND" H 7005 2527 50  0000 C CNN
+F 2 "" H 7000 2700 50  0001 C CNN
+F 3 "" H 7000 2700 50  0001 C CNN
+	1    7000 2700
+	-1   0    0    -1
+$EndComp
+Wire Wire Line
+	7000 4650 7000 4450
+Wire Wire Line
+	7000 4450 6400 4450
+Text GLabel 5400 1600 1    50   Input ~ 0
+v_load
+$Comp
+L Relay:G5LE-1 K1
+U 1 1 5FD31D61
+P 5600 2500
+F 0 "K1" H 5170 2454 50  0000 R CNN
+F 1 "G5LE-1" H 5170 2545 50  0000 R CNN
+F 2 "Relay_THT:Relay_SPDT_Omron-G5LE-1" H 6050 2450 50  0001 L CNN
+F 3 "http://www.omron.com/ecb/products/pdf/en-g5le.pdf" H 5600 2500 50  0001 C CNN
+	1    5600 2500
+	-1   0    0    1
+$EndComp
+Connection ~ 5800 2200
+Wire Wire Line
+	5300 2850 5300 2800
+Wire Wire Line
+	5800 2800 5800 2900
+Wire Wire Line
+	6400 1950 6400 2200
+Wire Wire Line
+	5400 2200 5400 1850
+Wire Wire Line
+	5400 1850 4900 1850
+Wire Wire Line
+	5400 1850 5400 1600
+Connection ~ 5400 1850
 $EndSCHEMATC

Commit message: Interface added
Parts:
- removed Q? (x2): 2N7002, Package_TO_SOT_SMD:SOT-23, symbol Transistor_FET:2N7002
- added Q? (x2): CJ3400, symbol Device:Q_NMOS_GDS
Connections:
- net GND: now also Q?.3 (S), Q?.3 (S)
- net at D?.2 (A), K2.5: now also Q?.2 (D)
- net at R?.1, R?.2: now also Q?.1 (G) (x2)
- net at D?.2 (A), K1.5: now also Q?.2 (D)
- net set_v renamed v_set
Changed lines of the file:
@@
 $EndDescr
 Text GLabel 1950 3400 0    50   Input ~ 0
-set_v
+v_set
 $Comp
 L Device:R R1
@@
 Wire Wire Line
 	5700 4450 6400 4450
-$Comp
-L Transistor_FET:2N7002 Q?
-U 1 1 60BD2568
-P 6500 3350
-F 0 "Q?" H 6705 3396 50  0000 L CNN
-F 1 "2N7002" H 6705 3305 50  0000 L CNN
-F 2 "Package_TO_SOT_SMD:SOT-23" H 6700 3275 50  0001 L CIN
-F 3 "https://www.fairchildsemi.com/datasheets/2N/2N7002.pdf" H 6500 3350 50  0001 L CNN
-	1    6500 3350
-	-1   0    0    -1
-$EndComp
-$Comp
-L Transistor_FET:2N7002 Q?
-U 1 1 60BE58B5
-P 6500 5600
-F 0 "Q?" H 6705 5646 50  0000 L CNN
-F 1 "2N7002" H 6705 5555 50  0000 L CNN
-F 2 "Package_TO_SOT_SMD:SOT-23" H 6700 5525 50  0001 L CIN
-F 3 "https://www.fairchildsemi.com/datasheets/2N/2N7002.pdf" H 6500 5600 50  0001 L CNN
-	1    6500 5600
-	-1   0    0    -1
-$EndComp
 NoConn ~ 5500 2800
 $Comp
@@
 	5400 1850 5400 1600
 Connection ~ 5400 1850
+$Comp
+L Device:Q_NMOS_GDS Q?
+U 1 1 60C76765
+P 6500 3350
+F 0 "Q?" H 6705 3396 50  0000 L CNN
+F 1 "CJ3400" H 6705 3305 50  0000 L CNN
+F 2 "" H 6700 3450 50  0001 C CNN
+F 3 "~" H 6500 3350 50  0001 C CNN
+	1    6500 3350
+	-1   0    0    -1
+$EndComp
+$Comp
+L Device:Q_NMOS_GDS Q?
+U 1 1 60C770C0
+P 6500 5600
+F 0 "Q?" H 6705 5646 50  0000 L CNN
+F 1 "CJ3400" H 6705 5555 50  0000 L CNN
+F 2 "" H 6700 5700 50  0001 C CNN
+F 3 "~" H 6500 5600 50  0001 C CNN
+	1    6500 5600
+	-1   0    0    -1
+$EndComp
 $EndSCHEMATC
