File: KiCad_DC_Load/Load_Circuit.sch (KiCad schematic (older format))
At the start: 38 parts, among them K1 G5LE-1, K2 G5LE-1, Q1 Q_NMOS_GDS, U1 LMC6482, U2 GS8552

Commit message: Some footprints assigned
Parts:
- removed D?: 1N4007, Diode_THT:D_DO-41_SOD81_P10.16mm_Horizontal, symbol Diode:1N4007
- removed Q?: CJ3400, symbol Device:Q_NMOS_GDS
- added D3: 1N4007WS, Diode_SMD:D_SOD-323, symbol Diode:1N4007
- added Q3: CJ3400, Package_TO_SOT_SMD:SOT-23, symbol Device:Q_NMOS_GSD
- C1, C2, C6, C7: renamed from C?; footprint (none) -> Capacitor_SMD:C_0805_2012Metric
- C3: renamed from C1; footprint (none) -> Capacitor_SMD:C_0805_2012Metric
- C4: renamed from C3; footprint (none) -> Capacitor_SMD:C_0805_2012Metric
- C5: renamed from C2; footprint (none) -> Capacitor_SMD:C_0805_2012Metric
- D2: renamed from D?; value 1N4007 -> 1N4007WS; footprint Diode_THT:D_DO-41_SOD81_P10.16mm_Horizontal -> Diode_SMD:D_SOD-323
- Q2: renamed from Q?; footprint (none) -> Package_TO_SOT_SMD:SOT-23; symbol Device:Q_NMOS_GDS -> Device:Q_NMOS_GSD
- R1, R2: footprint (none) -> Resistor_SMD:R_0805_2012Metric
- R10, R13, R18, R19, R20, R21: renamed from R?; footprint (none) -> Resistor_SMD:R_0805_2012Metric
- R12: renamed from R4; footprint (none) -> Resistor_SMD:R_0805_2012Metric
- R15: renamed from R5; footprint (none) -> Resistor_SMD:R_0805_2012Metric
- R3: renamed from R7; footprint (none) -> Resistor_SMD:R_0805_2012Metric
- R4: renamed from R14; footprint (none) -> Resistor_SMD:R_0805_2012Metric
- R5: renamed from R3; footprint (none) -> Resistor_SMD:R_0805_2012Metric
- R6: renamed from R15; footprint (none) -> Resistor_SMD:R_0805_2012Metric
- R7: renamed from R6; footprint (none) -> Resistor_SMD:R_0805_2012Metric
- R8: renamed from R13; footprint (none) -> Resistor_SMD:R_0805_2012Metric
- U1: renamed from U2; footprint (none) -> Package_SO:SOIC-8_3.9x4.9mm_P1.27mm
- U2: renamed from U1; footprint (none) -> Package_SO:SOIC-8_3.9x4.9mm_P1.27mm
- renumbered K2 to K1, K1 to K2, R9 to R11, R10 to R14, R11 to R16, R12 to R17, R8 to R9
Connections:
- net GND: now also C1.2, C2.2, Q2.2 (S), R15.1, Q3.2 (S); no longer Q2.3 (S)
- net v_9: now also D3.1 (K)
- net at K1.5: now also D3.2 (A), Q3.3 (D)
- net at R19.2, R21.1: now also Q3.1 (G)
- net at D2.2 (A), K2.5: now also Q2.3 (D); no longer Q2.2 (D)
Other:
- moved on the sheet: C2

Commit message: 10 pin connector footprint updated
Parts:
- R11, R14, R16, R9: footprint (none) -> Cement_resistor:R_Cement_Resistor_L22.2mm_W9.5mm_PS14.30mm_P25.40mm
- R17: footprint (none) -> Resistor_THT:R_Axial_DIN0516_L15.5mm_D5.0mm_P20.32mm_Horizontal
Changed lines of the file:
@@
 F 0 "R11" H 4620 5646 50  0000 L CNN
 F 1 "2" H 4620 5555 50  0000 L CNN
-F 2 "" V 4480 5600 50  0001 C CNN
+F 2 "Cement_resistor:R_Cement_Resistor_L22.2mm_W9.5mm_PS14.30mm_P25.40mm" V 4480 5600 50  0001 C CNN
 F 3 "~" H 4550 5600 50  0001 C CNN
 	1    4550 5600
@@
 F 0 "R9" H 4320 5646 50  0000 L CNN
 F 1 "2" H 4320 5555 50  0000 L CNN
-F 2 "" V 4180 5600 50  0001 C CNN
+F 2 "Cement_resistor:R_Cement_Resistor_L22.2mm_W9.5mm_PS14.30mm_P25.40mm" V 4180 5600 50  0001 C CNN
 F 3 "~" H 4250 5600 50  0001 C CNN
 	1    4250 5600
@@
 F 0 "R14" H 4920 5646 50  0000 L CNN
 F 1 "2" H 4920 5555 50  0000 L CNN
-F 2 "" V 4780 5600 50  0001 C CNN
+F 2 "Cement_resistor:R_Cement_Resistor_L22.2mm_W9.5mm_PS14.30mm_P25.40mm" V 4780 5600 50  0001 C CNN
 F 3 "~" H 4850 5600 50  0001 C CNN
 	1    4850 5600
@@
 F 0 "R16" H 5220 5646 50  0000 L CNN
 F 1 "2" H 5220 5555 50  0000 L CNN
-F 2 "" V 5080 5600 50  0001 C CNN
+F 2 "Cement_resistor:R_Cement_Resistor_L22.2mm_W9.5mm_PS14.30mm_P25.40mm" V 5080 5600 50  0001 C CNN
 F 3 "~" H 5150 5600 50  0001 C CNN
 	1    5150 5600
@@
 F 0 "R17" H 5570 5646 50  0000 L CNN
 F 1 "5.1" H 5570 5555 50  0000 L CNN
-F 2 "" V 5430 5600 50  0001 C CNN
+F 2 "Resistor_THT:R_Axial_DIN0516_L15.5mm_D5.0mm_P20.32mm_Horizontal" V 5430 5600 50  0001 C CNN
 F 3 "~" H 5500 5600 50  0001 C CNN
 	1    5500 5600
