File: KiCad_DC_Load/MCU.sch (KiCad schematic (older format))
At the start: 4 parts

Commit message: Some footprints assigned
Parts:
- R22, R24: renamed from R?; value R -> 4.7k; footprint (none) -> Resistor_SMD:R_0805_2012Metric
- R23: renamed from R?; footprint (none) -> Resistor_SMD:R_0805_2012Metric
- gave numbers to parts that had none: 1
Connections:
- no-connect marks 0 -> 23
Changed lines of the file:
@@
 Sheet 3 6
 Title "MCU"
-Date "2020-12-09"
-Rev ""
+Date "2021-06-16"
+Rev "v01"
 Comp ""
 Comment1 ""
 Comment2 ""
 Comment3 ""
-Comment4 "HappyDonuts"
+Comment4 "Author: HappyDonuts"
 $EndDescr
 $Comp
-L STM32_Dev_Boards:STM32F401CEU6 STM?
+L STM32_Dev_Boards:STM32F401CEU6 STM1
 U 1 1 60C66872
 P 5150 3850
-F 0 "STM?" H 5150 5515 50  0000 C CNN
+F 0 "STM1" H 5150 5515 50  0000 C CNN
 F 1 "STM32F401CEU6" H 5150 5424 50  0000 C CNN
 F 2 "" H 5200 4450 50  0001 C CNN
@@
 	4500 4700 4650 4700
 $Comp
-L Device:R R?
+L Device:R R22
 U 1 1 60C6AD5D
 P 5850 3600
-F 0 "R?" H 5920 3646 50  0000 L CNN
-F 1 "R" H 5920 3555 50  0000 L CNN
-F 2 "" V 5780 3600 50  0001 C CNN
+F 0 "R22" H 5920 3646 50  0000 L CNN
+F 1 "4.7k" H 5920 3555 50  0000 L CNN
+F 2 "Resistor_SMD:R_0805_2012Metric" V 5780 3600 50  0001 C CNN
 F 3 "~" H 5850 3600 50  0001 C CNN
 	1    5850 3600
@@
 $EndComp
 $Comp
-L Device:R R?
+L Device:R R24
 U 1 1 60C6B5EE
 P 6250 3600
-F 0 "R?" H 6320 3646 50  0000 L CNN
-F 1 "R" H 6320 3555 50  0000 L CNN
-F 2 "" V 6180 3600 50  0001 C CNN
+F 0 "R24" H 6320 3646 50  0000 L CNN
+F 1 "4.7k" H 6320 3555 50  0000 L CNN
+F 2 "Resistor_SMD:R_0805_2012Metric" V 6180 3600 50  0001 C CNN
 F 3 "~" H 6250 3600 50  0001 C CNN
 	1    6250 3600
@@
 $EndComp
 $Comp
-L power:GND #PWR?
+L power:GND #PWR017
 U 1 1 60C6BA05
-P 5850 3750
-F 0 "#PWR?" H 5850 3500 50  0001 C CNN
-F 1 "GND" H 5855 3577 50  0000 C CNN
-F 2 "" H 5850 3750 50  0001 C CNN
-F 3 "" H 5850 3750 50  0001 C CNN
-	1    5850 3750
-	1    0    0    -1
-$EndComp
-$Comp
-L power:GND #PWR?
+P 5850 3800
+F 0 "#PWR017" H 5850 3550 50  0001 C CNN
+F 1 "GND" H 5855 3627 50  0000 C CNN
+F 2 "" H 5850 3800 50  0001 C CNN
+F 3 "" H 5850 3800 50  0001 C CNN
+	1    5850 3800
+	1    0    0    -1
+$EndComp
+$Comp
+L power:GND #PWR018
 U 1 1 60C6C132
 P 6250 3750
-F 0 "#PWR?" H 6250 3500 50  0001 C CNN
+F 0 "#PWR018" H 6250 3500 50  0001 C CNN
 F 1 "GND" H 6255 3577 50  0000 C CNN
 F 2 "" H 6250 3750 50  0001 C CNN
@@
 	5850 2750 5650 2750
 $Comp
-L power:GND #PWR?
+L power:GND #PWR016
 U 1 1 60C74AC0
 P 5750 2600
-F 0 "#PWR?" H 5750 2350 50  0001 C CNN
+F 0 "#PWR016" H 5750 2350 50  0001 C CNN
 F 1 "GND" H 5850 2600 50  0000 C CNN
 F 2 "" H 5750 2600 50  0001 C CNN
@@
 	5650 2600 5750 2600
 $Comp
-L power:GND #PWR?
+L power:GND #PWR015
 U 1 1 60C76110
 P 4550 5150
-F 0 "#PWR?" H 4550 4900 50  0001 C CNN
+F 0 "#PWR015" H 4550 4900 50  0001 C CNN
 F 1 "GND" H 4450 5150 50  0000 C CNN
 F 2 "" H 4550 5150 50  0001 C CNN
@@
 	4550 5150 4650 5150
 $Comp
-L Device:R R?
+L Device:R R23
 U 1 1 60C76D58
 P 6000 4100
-F 0 "R?" V 5793 4100 50  0000 C CNN
+F 0 "R23" V 5793 4100 50  0000 C CNN
 F 1 "R" V 5884 4100 50  0000 C CNN
-F 2 "" V 5930 4100 50  0001 C CNN
+F 2 "Resistor_SMD:R_0805_2012Metric" V 5930 4100 50  0001 C CNN
 F 3 "~" H 6000 4100 50  0001 C CNN
 	1    6000 4100
@@
 Wire Wire Line
 	6150 4100 6300 4100
+NoConn ~ 5650 5300
+NoConn ~ 5650 5150
+NoConn ~ 5650 5000
+NoConn ~ 5650 4850
+NoConn ~ 5650 4700
+NoConn ~ 4650 4850
+NoConn ~ 4650 3950
+NoConn ~ 4650 3800
+NoConn ~ 4650 3650
+NoConn ~ 4650 3500
+NoConn ~ 4650 3350
+NoConn ~ 4650 3200
+NoConn ~ 4650 3050
+NoConn ~ 4650 2750
+NoConn ~ 4650 2600
+NoConn ~ 4650 2450
+NoConn ~ 5650 2900
+NoConn ~ 5650 3050
+NoConn ~ 5650 3500
+NoConn ~ 5650 3650
+NoConn ~ 5650 3800
+NoConn ~ 5650 3950
+NoConn ~ 4650 2900
+Wire Wire Line
+	5850 3800 5850 3750
 $EndSCHEMATC
